File: PWM_breakout_board/PWM_breakout_board.kicad_sch (KiCad schematic)
At the start: 8 parts, among them J1 Power, J2 Input, J3 Out 1, J4 Out 2, J5 Out 3, J6 Out 4

Commit message: Assigns footprints to symbols in PWM breakout board schematics
Parts:
- H1, H2: footprint (none) -> MountingHole:MountingHole_4.3mm_M4_ISO7380
- J1: footprint (none) -> TerminalBlock:TerminalBlock_bornier-2_P5.08mm
- J2: footprint (none) -> Connector_JST:JST_XH_B5B-XH-AM_1x05_P2.50mm_Vertical
- J3, J4, J5, J6: footprint (none) -> TerminalBlock:TerminalBlock_bornier-3_P5.08mm
Changed lines of the file:
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@@
       (effects (font (size 1.27 1.27)) (justify left))
     )
-    (property "Footprint" "" (at 210.82 91.44 0)
+    (property "Footprint" "TerminalBlock:TerminalBlock_bornier-3_P5.08mm" (at 210.82 91.44 0)
       (effects (font (size 1.27 1.27)) hide)
     )
@@
       (effects (font (size 1.27 1.27)) (justify left))
     )
-    (property "Footprint" "" (at 99.06 104.14 0)
+    (property "Footprint" "Connector_JST:JST_XH_B5B-XH-AM_1x05_P2.50mm_Vertical" (at 99.06 104.14 0)
       (effects (font (size 1.27 1.27)) hide)
     )
@@
       (effects (font (size 1.27 1.27)) (justify left))
     )
-    (property "Footprint" "" (at 185.42 91.44 0)
+    (property "Footprint" "TerminalBlock:TerminalBlock_bornier-3_P5.08mm" (at 185.42 91.44 0)
       (effects (font (size 1.27 1.27)) hide)
     )
@@
       (effects (font (size 1.27 1.27)) (justify left))
     )
-    (property "Footprint" "" (at 99.06 74.93 0)
+    (property "Footprint" "TerminalBlock:TerminalBlock_bornier-2_P5.08mm" (at 99.06 74.93 0)
       (effects (font (size 1.27 1.27)) hide)
     )
@@
       (effects (font (size 1.27 1.27)) (justify left))
     )
-    (property "Footprint" "" (at 160.02 91.44 0)
+    (property "Footprint" "TerminalBlock:TerminalBlock_bornier-3_P5.08mm" (at 160.02 91.44 0)
       (effects (font (size 1.27 1.27)) hide)
     )
@@
       (effects (font (size 1.27 1.27)) (justify left))
     )
-    (property "Footprint" "" (at 134.62 91.44 0)
+    (property "Footprint" "TerminalBlock:TerminalBlock_bornier-3_P5.08mm" (at 134.62 91.44 0)
       (effects (font (size 1.27 1.27)) hide)
     )
@@
       (effects (font (size 1.27 1.27)) (justify left))
     )
-    (property "Footprint" "" (at 34.29 34.29 0)
+    (property "Footprint" "MountingHole:MountingHole_4.3mm_M4_ISO7380" (at 34.29 34.29 0)
       (effects (font (size 1.27 1.27)) hide)
     )
@@
       (effects (font (size 1.27 1.27)) (justify left))
     )
-    (property "Footprint" "" (at 34.29 25.4 0)
-      (effects (font (size 1.27 1.27)) hide)
-    )
+    (property "Footprint" "MountingHole:MountingHole_4.3mm_M4_ISO7380" (at 34.29 25.4 0)
+      (effects (font (size 1.27 1.27)) hide)
+    )
