File: PWM_breakout_board/PWM_breakout_board.kicad_pcb (KiCad board)
At the start: 2 copper layers, 100 x 40 mm, 9 parts, among them J1 Power, J2 Input, J3 Out 1, J4 Out 2, J5 Out 3, J6 Out 4

Commit message: Adds personal logo do PWM breakout board
Parts:
- added Ref**: Val**, AmieiroFootprints:ipe_logo_FSilk_10x10, F.Cu at (88.0, 82.0)

Commit message: Adds silkscreen to outputs in breakout board
Other:
- board text added: "+"
- board text added: "-"
- board text added: "1"
- board text added: "2"
- board text added: "3"
- board text added: "4"
- board text added: "data"
Changed lines of the file:
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@@
+    (effects (font (size 1.5 1.5) (thickness 0.3) bold) (justify left bottom))
+  )
+  (gr_text "data" (at 163 108.1) (layer "F.SilkS")
+    (effects (font (size 1 1) (thickness 0.15)) (justify left bottom))
+  )
+  (gr_text "1" (at 83.6 104.4) (layer "F.SilkS")
+    (effects (font (size 2 2) (thickness 0.3)) (justify left bottom))
+  )
+  (gr_text "data" (at 116 108.1) (layer "F.SilkS")
+    (effects (font (size 1 1) (thickness 0.15)) (justify left bottom))
+  )
+  (gr_text "data" (at 139.6 108.1) (layer "F.SilkS")
+    (effects (font (size 1 1) (thickness 0.15)) (justify left bottom))
+  )
+  (gr_text "data" (at 92.4 108.2) (layer "F.SilkS")
+    (effects (font (size 1 1) (thickness 0.15)) (justify left bottom))
+  )
+  (gr_text "2" (at 107 104.4) (layer "F.SilkS")
+    (effects (font (size 2 2) (thickness 0.3)) (justify left bottom))
+  )
+  (gr_text "-" (at 98.2 108.5) (layer "F.SilkS")
+    (effects (font (size 1.5 1.5) (thickness 0.3) bold) (justify left bottom))
+  )
+  (gr_text "4" (at 154.2 104.4) (layer "F.SilkS")
+    (effects (font (size 2 2) (thickness 0.3)) (justify left bottom))
+  )
+  (gr_text "-" (at 121.8 108.4) (layer "F.SilkS")
+    (effects (font (size 1.5 1.5) (thickness 0.3) bold) (justify left bottom))
+  )
+  (gr_text "-" (at 145.4 108.4) (layer "F.SilkS")
+    (effects (font (size 1.5 1.5) (thickness 0.3) bold) (justify left bottom))
+  )
+  (gr_text "+" (at 158.319857 108.4) (layer "F.SilkS")
+    (effects (font (size 1.5 1.5) (thickness 0.3) bold) (justify left bottom))
+  )
+  (gr_text "+" (at 87.719857 108.5) (layer "F.SilkS")
+    (effects (font (size 1.5 1.5) (thickness 0.3) bold) (justify left bottom))
+  )
+  (gr_text "+" (at 134.919857 108.4) (layer "F.SilkS")
+    (effects (font (size 1.5 1.5) (thickness 0.3) bold) (justify left bottom))
+  )
+  (gr_text "+" (at 111.319857 108.4) (layer "F.SilkS")
+    (effects (font (size 1.5 1.5) (thickness 0.3) bold) (justify left bottom))
+  )
+  (gr_text "3" (at 130.4 104.4) (layer "F.SilkS")
+    (effects (font (size 2 2) (thickness 0.3)) (justify left bottom))
+  )
+  (gr_text "-" (at 168.8 108.4) (layer "F.SilkS")
     (effects (font (size 1.5 1.5) (thickness 0.3) bold) (justify left bottom))
   )

Commit message: Generates gerber files for splitter
Other:
- board text added: "Input"
- board text added: "Power"
Changed lines of the file:
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@@
       (outputformat 1)
       (mirror false)
-      (drillshape 1)
+      (drillshape 0)
       (scaleselection 1)
-      (outputdirectory "")
+      (outputdirectory "Gerber/")
     )
   )
@@
   (footprint "AmieiroFootprints:ipe_logo_FSilk_10x10" (layer "F.Cu")
     (at 88 82)
-    (attr through_hole)
+    (attr through_hole board_only)
     (fp_text reference "Ref**" (at 0 0) (layer "F.SilkS") hide
         (effects (font (size 1.27 1.27) (thickness 0.15)))
@@
     )
   )
+  (gr_line (start 137.4 72.2) (end 124.8 72.2)
+    (stroke (width 0.15) (type default)) (layer "F.SilkS"))
+  (gr_line (start 95.8 78.8) (end 95.8 71.2)
+    (stroke (width 0.15) (type default)) (layer "F.SilkS"))
+  (gr_line (start 122.6 75.2) (end 122.6 76.6)
+    (stroke (width 0.15) (type default)) (layer "F.SilkS"))
+  (gr_line (start 123.6 75.2) (end 123.6 74)
+    (stroke (width 0.15) (type default)) (layer "F.SilkS"))
+  (gr_line (start 122.6 77.8) (end 122.6 71.6)
+    (stroke (width 0.15) (type default)) (layer "F.SilkS"))
+  (gr_line (start 124.8 76.6) (end 124.8 77.8)
+    (stroke (width 0.15) (type default)) (layer "F.SilkS"))
+  (gr_line (start 106.2 78.8) (end 95.8 78.8)
+    (stroke (width 0.15) (type default)) (layer "F.SilkS"))
+  (gr_line (start 122.6 71.6) (end 123 71.6)
+    (stroke (width 0.15) (type default)) (layer "F.SilkS"))
+  (gr_line (start 137.4 75.2) (end 137.4 72.2)
+    (stroke (width 0.15) (type default)) (layer "F.SilkS"))
+  (gr_line (start 138.4 75.2) (end 137.4 75.2)
+    (stroke (width 0.15) (type default)) (layer "F.SilkS"))
+  (gr_line (start 106.2 72.4) (end 95.8 72.4)
+    (stroke (width 0.15) (type default)) (layer "F.SilkS"))
+  (gr_line (start 106.2 71.2) (end 106.2 78.8)
+    (stroke (width 0.15) (type default)) (layer "F.SilkS"))
+  (gr_line (start 136.4 77.8) (end 136.4 76.6)
+    (stroke (width 0.15) (type default)) (layer "F.SilkS"))
+  (gr_line (start 138.4 77.8) (end 122.6 77.8)
+    (stroke (width 0.15) (type default)) (layer "F.SilkS"))
+  (gr_line (start 123.6 75.2) (end 122.6 75.2)
+    (stroke (width 0.15) (type default)) (layer "F.SilkS"))
+  (gr_line (start 123 71.6) (end 138.4 71.6)
+    (stroke (width 0.15) (type default)) (layer "F.SilkS"))
+  (gr_line (start 136.4 76.6) (end 138.4 76.6)
+    (stroke (width 0.15) (type default)) (layer "F.SilkS"))
+  (gr_line (start 96 72.4) (end 106.2 72.4)
+    (stroke (width 0.15) (type default)) (layer "F.SilkS"))
+  (gr_line (start 138.4 71.6) (end 138.4 77.8)
+    (stroke (width 0.15) (type default)) (layer "F.SilkS"))
+  (gr_line (start 95.8 71.2) (end 106.2 71.2)
+    (stroke (width 0.15) (type default)) (layer "F.SilkS"))
+  (gr_line (start 122.6 76.6) (end 124.8 76.6)
+    (stroke (width 0.15) (type default)) (layer "F.SilkS"))
   (gr_line locked (start 179.964466 99.928932) (end 180.035534 80)
     (stroke (width 0.1) (type default)) (layer "Edge.Cuts"))
@@
     (effects (font (size 1.5 1.5) (thickness 0.3) bold) (justify left bottom))
   )
+  (gr_text "Power" (at 106.6 75.6) (layer "F.SilkS")
+    (effects (font (size 1 1) (thickness 0.15)) (justify left bottom))
+  )
   (gr_text "+" (at 134.919857 108.4) (layer "F.SilkS")
     (effects (font (size 1.5 1.5) (thickness 0.3) bold) (justify left bottom))
   )
+  (gr_text "Input" (at 140 75.6) (layer "F.SilkS")
+    (effects (font (size 1 1) (thickness 0.15)) (justify left bottom))
+  )
   (gr_text "+" (at 111.319857 108.4) (layer "F.SilkS")
     (effects (font (size 1.5 1.5) (thickness 0.3) bold) (justify left bottom))
@@
     (effects (font (size 1.5 1.5) (thickness 0.3) bold) (justify left bottom))
   )
-  (dimension (type aligned) (layer "F.Cu")
+  (dimension (type aligned) (layer "User.1")
     (pts (xy 80 70) (xy 180 70))
     (height -7)
-    (gr_text "100,0000 mm" (at 130 61.2) (layer "F.Cu")
+    (gr_text "100,0000 mm" (at 130 61.2) (layer "User.1")
       (effects (font (size 1.5 1.5) (thickness 0.3)))
     )
